Commit message: Hamer_mini v0.2
ChangeLog v0.2 -- 29.01.2020
--Ultrasonic sensors added.
Requirements:
In order for the sensors to work properly, "gazebo_ros_pkgs" files must be downloaded.
$ cd ~/hamer_mini/src
$ git clone https://github.com/ros-simulation/gazebo_ros_pkgs.git -b melodic-devel

File: hamer_mini/urdf/hamer_mini.urdf (robot description, URDF)
Before this commit: robot hamer_mini, 6 links, 5 joints
Links:
- added link sonar_back, mass 1e-5; collision box size=0.001 0.001 0.001; visual box size=0.001 0.001 0.001
- added link sonar_front, mass 1e-5; collision box size=0.001 0.001 0.001; visual box size=0.001 0.001 0.001
- added link sonar_left, mass 1e-5; collision box size=0.001 0.001 0.001; visual box size=0.001 0.001 0.001
- added link sonar_right, mass 1e-5; collision box size=0.001 0.001 0.001; visual box size=0.001 0.001 0.001
Joints:
- added joint sonar_back_joint: type fixed, parent base_link, child sonar_back, origin xyz=-0.1275 0 0.01 rpy=0 3.14 0, axis 0 0 0
- added joint sonar_front_joint: type fixed, parent base_link, child sonar_front, origin xyz=0.1275 0 0.01 rpy=0 0 0, axis 0 0 0
- added joint sonar_left_joint: type fixed, parent base_link, child sonar_left, origin xyz=0 0.075 0.01 rpy=0 0 1.57, axis 0 0 0
- added joint sonar_right_joint: type fixed, parent base_link, child sonar_right, origin xyz=0 -0.075 0.01 rpy=0 0 -1.57, axis 0 0 0

Commit message: Hamer_mini v0.3
Changelog v0.3 (31-01-2020)
- Added "gazebo_ros_control" to hamer_mini's urdf file.
- Changed ultrasonic sensors positions and quantities.

File: hamer_mini/urdf/hamer_mini.urdf (robot description, URDF)
Before this commit: robot hamer_mini, 10 links, 9 joints
Links:
- removed link sonar_back
Joints:
- removed joint sonar_back_joint
- joint sonar_left_joint: origin xyz=0 0.075 0.01 rpy=0 0 1.57 -> xyz=0.1275 0.075 0.01 rpy=0 0 0.785
- joint sonar_right_joint: origin xyz=0 -0.075 0.01 rpy=0 0 -1.57 -> xyz=0.1275 -0.075 0.01 rpy=0 0 -0.785

Commit message: HAMER_mini v0.4 - (01-02-2020)
Changelog v0.4
-Available SLAM package usage.
-Added laser sensor.
-Available mapping with laser sensor to gazebo maps.

File: hamer_mini/urdf/hamer_mini.urdf (robot description, URDF)
Before this commit: robot hamer_mini, 9 links, 8 joints
Links:
- removed link sonar_front
- added link hokuyo_link; collision cylinder length=0.04 radius=0.02; visual cylinder length=0.04 radius=0.02
- added link sonar_back, mass 1e-5; collision box size=0.001 0.001 0.001; visual box size=0.001 0.001 0.001
Joints:
- removed joint sonar_front_joint
- added joint hokuyo_joint: type fixed, parent base_link, child hokuyo_link, origin xyz=0.1 0 0.04 rpy=0 0 0, axis 0 1 0
- added joint sonar_back_joint: type fixed, parent base_link, child sonar_back, origin xyz=-0.1275 0 0.01 rpy=0 3.14 0, axis 0 0 0

Commit message: Add files via upload

File: hamer_mini/urdf/hamer_mini.urdf (robot description, URDF)
Before this commit: robot hamer_mini, 10 links, 9 joints
Links:
- removed link dummy
- removed link hokuyo_link
- added link camera_link, mass 1e-5; collision box size=0.02 0.05 0.015; visual mesh filename=package://hamer_mini/meshes/Stl/Intel_RealSense_Depth_Camer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 scale=0.00105 0.00105 0.00105
- added link laser_platform_link, mass 0.01; collision cylinder length=0.04 radius=0.01; visual cylinder length=0.04 radius=0.01
- added link tfmini_link; collision box size=0.042 0.015 0.016; visual box size=0.015 0.042 0.016
- link base_link: geometry collision box size=0.255 0.150 0.04; visual mesh filename=package://hamer_mini/meshes/Stl/base_link.STL
- link left_back_wheel: geometry collision cylinder length=0.026 radius=0.0325; visual mesh filename=package://hamer_mini/meshes/Stl/left_back_wheel.STL
- link left_front_wheel: geometry collision cylinder length=0.026 radius=0.0325; visual mesh filename=package://hamer_mini/meshes/Stl/left_front_wheel.STL
- link right_back_wheel: geometry collision cylinder length=0.026 radius=0.0325; visual mesh filename=package://hamer_mini/meshes/Stl/right_back_wheel.STL
- link right_front_wheel: geometry collision cylinder length=0.026 radius=0.0325; visual mesh filename=package://hamer_mini/meshes/Stl/right_front_wheel.STL
Joints:
- removed joint dummy_joint
- removed joint hokuyo_joint
- added joint camera_joint: type fixed, parent base_link, child camera_link, origin xyz=0.1275 0 0.028 rpy=0 0 0, axis 0 1 0
- added joint joint_laser_platform_link: type fixed, parent base_link, child laser_platform_link, origin xyz=-0.05 0 0.04 rpy=0 0 0, axis 0 1 0
- added joint tfmini_joint: type fixed, parent base_link, child tfmini_link, origin xyz=-0.05 0 0.07 rpy=0 0 0, axis 0 1 0

Commit message: Version v0.5.2 Minor Update

File: hamer_mini/urdf/hamer_mini.urdf (robot description, URDF)
Before this commit: robot hamer_mini, 11 links, 10 joints
Links:
- added link dummy
Joints:
- added joint dummy_joint: type fixed, parent dummy, child base_link
- joint joint_left_back_wheel: origin xyz=-0.07 0.086 0 rpy=0 0 0 -> xyz=-0.06 0.08 0.011 rpy=0 0 0
- joint joint_left_front_wheel: origin xyz=0.07 0.086 0 rpy=0 0 0 -> xyz=0.06 0.08 0.011 rpy=0 0 0
- joint joint_right_back_wheel: origin xyz=-0.07 -0.086 0 rpy=0 0 0 -> xyz=-0.06 -0.08 0.011 rpy=0 0 0
- joint joint_right_front_wheel: origin xyz=0.07 -0.086 0 rpy=0 0 0 -> xyz=0.06 -0.08 0.011 rpy=0 0 0
